Commit message: Add rplidar udev

File: urdf/rosgolf.urdf (robot description, URDF)
Before this commit: robot ugv, 4 links, 3 joints
Links:
- removed link base_footprint
- removed link imu
- removed link laser
- added link cover; visual box size=0.72 0.485 0.15
- added link fwheel; visual cylinder length=0.02 radius=0.035
- added link lwheel; visual cylinder length=0.07 radius=0.12
- added link rwheel; visual cylinder length=0.07 radius=0.12
- added link scanner; visual cylinder length=0.04 radius=0.04
- link base_link: mass 1.0 -> None; geometry visual box size=0.72 0.485 0.05
Joints:
- removed joint base_footprint_joint
- removed joint imu_link_joint
- removed joint laser_frame_link_joint
- added joint base_to_fwheel: type fixed, parent base_link, child fwheel, origin xyz=0.47 0 0.035 rpy=0 0 0
- added joint base_to_lwheel: type fixed, parent base_link, child lwheel, origin xyz=0 0.29 0.12 rpy=1.5708 0 0
- added joint base_to_rwheel: type fixed, parent base_link, child rwheel, origin xyz=0 -0.29 0.12 rpy=-1.5708 0 0
- added joint base_to_scanner: type fixed, parent base_link, child scanner, origin xyz=0.0 0 0.26 rpy=0 0 0

Commit message: Add rplidar udev

File: urdf/rosgolf.urdf (robot description, URDF)
Before this commit: robot rosgolf_robot, 6 links, 4 joints
Joints:
- added joint base_to_cover: type fixed, parent base_link, child cover, origin xyz=0 0 0 rpy=0 0 0

Commit message: Add rplidar udev

File: urdf/rosgolf.urdf (robot description, URDF)
Before this commit: robot rosgolf_robot, 6 links, 5 joints
Links:
- removed link scanner
- added link laser; visual cylinder length=0.04 radius=0.04
Joints:
- joint base_to_scanner: child scanner -> laser

Commit message: Add rplidar udev

File: urdf/rosgolf.urdf (robot description, URDF)
Before this commit: robot rosgolf_robot, 7 links, 6 joints
Links:
- link base_link: geometry collision box size=0.72 0.485 0.05; visual box size=0.72 0.485 0.05

Commit message: Add rplidar udev

File: urdf/rosgolf.urdf (robot description, URDF)
Before this commit: robot rosgolf_robot, 7 links, 6 joints
Links:
- link base_link: geometry collision box size=0.72 0.485 0.35; visual box size=0.72 0.485 0.05

Commit message: Add rplidar udev

File: urdf/rosgolf.urdf (robot description, URDF)
Before this commit: robot rosgolf_robot, 7 links, 6 joints
Links:
- link base_link: geometry collision box size=0.72 0.485 0.40; visual box size=0.72 0.485 0.05

Commit message: URDF

File: urdf/rosgolf.urdf (robot description, URDF)
Before this commit: robot rosgolf_robot, 7 links, 6 joints
Links:
- link base_link: geometry collision box size=0.72 0.70 0.40; visual box size=0.72 0.485 0.05

Commit message: Odometry

File: urdf/rosgolf.urdf (robot description, URDF)
Before this commit: robot rosgolf_robot, 7 links, 6 joints
Joints:
- joint base_footprint_joint: child base_link -> base_footprint; parent base_footprint -> base_link

Commit message: Odometry

File: urdf/rosgolf.urdf (robot description, URDF)
Before this commit: robot rosgolf_robot, 7 links, 6 joints
Joints:
- removed joint base_to_lwheel
- removed joint base_to_rwheel
- added joint left_wheel_hinge: type fixed, parent base_link, child lwheel, origin xyz=0 0.29 0.12 rpy=1.5708 0 0
- added joint right_wheel_hinge: type fixed, parent base_link, child rwheel, origin xyz=0 -0.29 0.12 rpy=-1.5708 0 0

Commit message: Odometry

File: urdf/rosgolf.urdf (robot description, URDF)
Before this commit: robot rosgolf_robot, 7 links, 6 joints
Joints:
- joint left_wheel_hinge: origin xyz=0 0.29 0.12 rpy=1.5708 0 0 -> xyz=0 0.29 0.12 rpy=0 0 0; type fixed -> continuous
- joint right_wheel_hinge: origin xyz=0 -0.29 0.12 rpy=-1.5708 0 0 -> xyz=0 -0.29 0.12 rpy=0 0 0; type fixed -> continuous

Commit message: Odometry

File: urdf/rosgolf.urdf (robot description, URDF)
Before this commit: robot rosgolf_robot, 7 links, 6 joints
Joints:
- joint left_wheel_hinge: axis (none) -> 0 1 0; origin xyz=0 0.29 0.12 rpy=0 0 0 -> xyz=0 0.29 0.12 rpy= 0 0
- joint right_wheel_hinge: axis (none) -> 0 1 0; origin xyz=0 -0.29 0.12 rpy=0 0 0 -> xyz=0 -0.29 0.12 rpy=-1.5708 0 0

Commit message: Odometry

File: urdf/rosgolf.urdf (robot description, URDF)
Before this commit: robot rosgolf_robot, 7 links, 6 joints
Joints:
- joint left_wheel_hinge: axis 0 1 0 -> 1 0 0
- joint right_wheel_hinge: axis 0 1 0 -> 1 0 0

Commit message: Odometry

File: urdf/rosgolf.urdf (robot description, URDF)
Before this commit: robot rosgolf_robot, 7 links, 6 joints
Joints:
- joint left_wheel_hinge: axis 1 0 0 -> (none)
- joint right_wheel_hinge: axis 1 0 0 -> (none)

Commit message: Odometry

File: urdf/rosgolf.urdf (robot description, URDF)
Before this commit: robot rosgolf_robot, 7 links, 6 joints
Joints:
- joint left_wheel_hinge: origin xyz=0 0.29 0.12 rpy= 0 0 -> xyz=0 0.29 0.12 rpy=0 0 0

Commit message: Odometry

File: urdf/rosgolf.urdf (robot description, URDF)
Before this commit: robot rosgolf_robot, 7 links, 6 joints
Joints:
- joint left_wheel_hinge: origin xyz=0 0.29 0.12 rpy=0 0 0 -> xyz=0 0.29 0.12 rpy=1.5708 0 0

Commit message: Odometry

File: urdf/rosgolf.urdf (robot description, URDF)
Before this commit: robot rosgolf_robot, 7 links, 6 joints
Links:
- link base_footprint: geometry visual cylinder length=0.07 radius=0.12

Commit message: Odometry

File: urdf/rosgolf.urdf (robot description, URDF)
Before this commit: robot rosgolf_robot, 6 links, 5 joints
Links:
- added link base_footprint; visual cylinder length=0.07 radius=0.12
Joints:
- added joint base_footprint_joint: type fixed, parent base_link, child base_footprint, origin xyz=0 0 0 rpy=0 0 0

Commit message: Params

File: urdf/rosgolf.urdf (robot description, URDF)
Before this commit: robot rosgolf_robot, 6 links, 5 joints
Links:
- added link base_footprint; visual cylinder length=0.01 radius=0.12
Joints:
- added joint base_footprint_joint: type fixed, parent base_footprint, child base_link, origin xyz=0 0 0 rpy=0 0 0

Commit message: Params

File: urdf/rosgolf.urdf (robot description, URDF)
Before this commit: robot rosgolf_robot, 7 links, 6 joints
Joints:
- joint left_wheel_hinge: axis (none) -> 0 0 1
- joint right_wheel_hinge: axis (none) -> 0 0 1

Commit message: Odometry

File: urdf/rosgolf.urdf (robot description, URDF)
Before this commit: robot rosgolf_robot, 6 links, 5 joints
Joints:
- joint base_to_scanner: origin xyz=0.0 0 0.26 rpy=0 0 0 -> xyz=0.0 -0.04 0.26 rpy=0 0 0

Commit message: Odometry

File: urdf/rosgolf.urdf (robot description, URDF)
Before this commit: robot rosgolf_robot, 6 links, 5 joints
Links:
- added link camera_odom_frame
Joints:
- added joint base_to_camera: type fixed, parent base_link, child camera_odom_frame, origin xyz=0.48 -0.045 0.145 rpy=0 0 0

Commit message: WebUI

File: urdf/rosgolf.urdf (robot description, URDF)
Before this commit: robot rosgolf_robot, 7 links, 6 joints
Links:
- added link sonar
Joints:
- added joint base_to_sonar: type fixed, parent base_link, child camera_odom_frame, origin xyz=0.48 0.0 0.145 rpy=0 0 0

Commit message: WebUI

File: urdf/rosgolf.urdf (robot description, URDF)
Before this commit: robot rosgolf_robot, 8 links, 7 joints
Joints:
- joint base_to_sonar: child camera_odom_frame -> sonar

Commit message: WebUI

File: urdf/rosgolf.urdf (robot description, URDF)
Before this commit: robot rosgolf_robot, 8 links, 7 joints
Links:
- added link imu
Joints:
- added joint imu_to_sonar: type fixed, parent base_link, child sonar, origin xyz=0.10 -10.0 0.18 rpy=0 0 0

Commit message: WebUI

File: urdf/rosgolf.urdf (robot description, URDF)
Before this commit: robot rosgolf_robot, 9 links, 8 joints
Joints:
- joint imu_to_sonar: child sonar -> imu

Commit message: IMU testing

File: urdf/rosgolf.urdf (robot description, URDF)
Before this commit: robot rosgolf_robot, 9 links, 8 joints
Joints:
- joint imu_to_sonar: origin xyz=0.10 -10.0 0.18 rpy=0 0 0 -> xyz=0.10 -0.10 0.18 rpy=0 0 0
